Commit message: fix size

File: urdf/sink_old.urdf (robot description, URDF)
Before this commit: robot sink, 5 links, 4 joints
Links:
- removed link fconnp2
Joints:
- removed joint press2
- joint press: origin xyz=50e-3 0 30e-3 rpy=0 -1.1 0 -> xyz=60e-3 0 5e-3 rpy=0 -1.1 0
- joint to_female: origin xyz=0 -140e-3 135e-3 rpy=3.14 1.57 -1.57 -> xyz=0 -120e-3 150e-3 rpy=3.14 1.57 -1.57
